File: kicad/riotee-solar-shield.kicad_sch (KiCad schematic)
At the start: 7 parts, among them J1 Conn_01x10, J2 Conn_01x12, SW1 SW_DIP_x02

Commit message: add MPNs in schematics
Parts:
- J1: MPN (none) -> PH1-10-UA
- J2: MPN (none) -> PH1-12-UA
- SC1, SC2, SC3, SC4: MPN (none) -> KXOB25-05X3F-TR
- SW1: MPN (none) -> ADE02S04
Changed lines of the file:
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@@
+      (effects (font (size 1.27 1.27)) hide)
+    )
+    (property "MPN" "KXOB25-05X3F-TR" (id 4) (at 172.72 105.41 0)
       (effects (font (size 1.27 1.27)) hide)
     )
@@
       (effects (font (size 1.27 1.27)) hide)
     )
+    (property "MPN" "KXOB25-05X3F-TR" (id 4) (at 129.54 105.41 0)
+      (effects (font (size 1.27 1.27)) hide)
+    )
     (pin "1")
     (pin "2")
@@
     )
     (property "Datasheet" "https://waf-e.dubudisk.com/anysolar.dubuplus.com/techsupport@anysolar.biz/O18Ae07/DubuDisk/www/Gen3/KXOB25-05X3F%20DATA%20SHEET%20202007.pdf" (id 3) (at 111.76 118.11 0)
+      (effects (font (size 1.27 1.27)) hide)
+    )
+    (property "MPN" "KXOB25-05X3F-TR" (id 4) (at 107.95 105.41 0)
       (effects (font (size 1.27 1.27)) hide)
     )
@@
       (effects (font (size 1.27 1.27)) hide)
     )
+    (property "MPN" "PH1-12-UA" (id 4) (at 177.8 55.88 0)
+      (effects (font (size 1.27 1.27)) hide)
+    )
     (pin "1")
     (pin "10")
@@
     )
     (property "Datasheet" "~" (id 3) (at 182.88 97.79 0)
+      (effects (font (size 1.27 1.27)) hide)
+    )
+    (property "MPN" "ADE02S04" (id 4) (at 182.88 97.79 0)
       (effects (font (size 1.27 1.27)) hide)
     )
@@
       (effects (font (size 1.27 1.27)) hide)
     )
+    (property "MPN" "PH1-10-UA" (id 4) (at 124.46 53.34 0)
+      (effects (font (size 1.27 1.27)) hide)
+    )
     (pin "1")
     (pin "10")
@@
       (effects (font (size 1.27 1.27)) hide)
     )
+    (property "MPN" "KXOB25-05X3F-TR" (id 4) (at 151.13 105.41 0)
+      (effects (font (size 1.27 1.27)) hide)
+    )

Commit message: add conformity marks and refine BOM
Changed lines of the file:
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@@
+    (stroke (width 0) (type default) (color 0 0 0 0))
+  )
+  (wire (pts (xy 208.28 69.85) (xy 208.28 73.66))
     (stroke (width 0) (type default) (color 0 0 0 0))
   )
@@
     )
     (property "Datasheet" "" (id 3) (at 170.18 73.66 0)
+      (effects (font (size 1.27 1.27)) hide)
+    )
+    (pin "1")
+  )
+  (symbol (lib_id "power:GND") (at 208.28 73.66 0) (unit 1)
+    (in_bom yes) (on_board yes) (fields_autoplaced)
+    (property "Reference" "#PWR04" (id 0) (at 208.28 80.01 0)
+      (effects (font (size 1.27 1.27)) hide)
+    )
+    (property "Value" "GND" (id 1) (at 208.28 78.1034 0))
+    (property "Footprint" "" (id 2) (at 208.28 73.66 0)
+      (effects (font (size 1.27 1.27)) hide)
+    )
+    (property "Datasheet" "" (id 3) (at 208.28 73.66 0)
       (effects (font (size 1.27 1.27)) hide)
     )
@@
     (pin "1")
   )
+  (symbol (lib_id "power:PWR_FLAG") (at 208.28 69.85 0) (unit 1)
+    (in_bom yes) (on_board yes) (fields_autoplaced)
+    (property "Reference" "#FLG01" (id 0) (at 208.28 67.945 0)
+      (effects (font (size 1.27 1.27)) hide)
+    )
+    (property "Value" "PWR_FLAG" (id 1) (at 208.28 66.2742 0))
+    (property "Footprint" "" (id 2) (at 208.28 69.85 0)
+      (effects (font (size 1.27 1.27)) hide)
+    )
+    (property "Datasheet" "~" (id 3) (at 208.28 69.85 0)
+      (effects (font (size 1.27 1.27)) hide)
+    )
+    (pin "1")
+  )
   (symbol (lib_id "power:GND") (at 107.95 113.03 0) (unit 1)
     (in_bom yes) (on_board yes) (fields_autoplaced)
@@
   )
   (symbol_instances
+    (path "/adf08bd8-0f4c-4945-ae89-38df52b687c9"
+      (reference "#FLG01") (unit 1) (value "PWR_FLAG") (footprint "")
+    )
     (path "/bb10caac-ce87-46e8-b982-dc38c18239db"
       (reference "#PWR01") (unit 1) (value "GND") (footprint "")
@@
       (reference "#PWR03") (unit 1) (value "GND") (footprint "")
     )
+    (path "/56773f75-ceb7-48f0-90eb-27534873d55c"
+      (reference "#PWR04") (unit 1) (value "GND") (footprint "")
+    )
     (path "/d4b3a3d6-6061-4cb8-beec-faff348cf04b"
