File: kicad/riotee-solar-shield.kicad_pcb (KiCad board)
At the start: 2 copper layers, 55.9 x 25.4 mm, 7 parts, among them J1 Conn_01x10, J2 Conn_01x12, SW1 SW_DIP_x02

Commit message: add kikit configuration for production panel
Parts:
- added REF**: Tab, riotee:KikitTab, F.Cu at (187.6, 75.2)
- added REF**: Tab, riotee:KikitTab, F.Cu at (187.6, 49.3)
- added REF**: Tab, riotee:KikitTab, F.Cu at (223.9, 50.5)
- added REF**: Tab, riotee:KikitTab, F.Cu at (233.9, 62.2)
- added REF**: Tab, riotee:KikitTab, F.Cu at (177.6, 62.2)
- added REF**: Tab, riotee:KikitTab, F.Cu at (223.9, 73.9)
Changed lines of the file:
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@@
     (pad_to_mask_clearance 0)
     (pcbplotparams
-      (layerselection 0x00010f8_ffffffff)
+      (layerselection 0x00010d8_ffffffff)
       (plot_on_all_layers_selection 0x0000000_00000000)
       (disableapertmacros false)
@@
   (net 21 "Net-(SC1-+)")
   (net 22 "Net-(SC4-+)")
+  (footprint "riotee:KikitTab" (layer "F.Cu")
+    (at 187.62 75.18 90)
+    (descr "A symbol representing annotation for tab placement")
+    (attr exclude_from_pos_files exclude_from_bom)
+    (fp_text reference "REF**" (at 0 -2 90) (layer "F.SilkS") hide
+        (effects (font (size 1 1) (thickness 0.15)))
+    )
+    (fp_text value "Tab" (at -2.75 -1 90) (layer "Dwgs.User")
+        (effects (font (size 1.2 1.2) (thickness 0.2)))
+    )
+    (fp_text user "KIKIT: width: 3mm" (at -5.5 0) (layer "Dwgs.User")
+        (effects (font (size 1 1) (thickness 0.15)))
+    )
+    (fp_line (start 0.25 0) (end -2.75 0)
+      (stroke (width 0.3) (type solid)) (layer "Dwgs.User"))
+    (fp_line (start 0.25 0) (end -0.75 -1)
+      (stroke (width 0.3) (type solid)) (layer "Dwgs.User"))
+    (fp_line (start 0.25 0) (end -0.75 1)
+      (stroke (width 0.3) (type solid)) (layer "Dwgs.User"))
+    (fp_line (start 0.25 1) (end 0.25 -1)
+      (stroke (width 0.3) (type solid)) (layer "Dwgs.User"))
+  )
   (footprint "riotee:AS_KXOB25_23x08" (layer "F.Cu")
     (at 215.4 66.548)
@@
     )
   )
+  (footprint "riotee:KikitTab" (layer "F.Cu")
+    (at 187.62 49.28 -90)
+    (descr "A symbol representing annotation for tab placement")
+    (attr exclude_from_pos_files exclude_from_bom)
+    (fp_text reference "REF**" (at 0 -2 90) (layer "F.SilkS") hide
+        (effects (font (size 1 1) (thickness 0.15)))
+    )
+    (fp_text value "Tab" (at -2.75 -1 90) (layer "Dwgs.User")
+        (effects (font (size 1.2 1.2) (thickness 0.2)))
+    )
+    (fp_text user "KIKIT: width: 3mm" (at -5.5 0) (layer "Dwgs.User")
+        (effects (font (size 1 1) (thickness 0.15)))
+    )
+    (fp_line (start 0.25 0) (end -2.75 0)
+      (stroke (width 0.3) (type solid)) (layer "Dwgs.User"))
+    (fp_line (start 0.25 0) (end -0.75 -1)
+      (stroke (width 0.3) (type solid)) (layer "Dwgs.User"))
+    (fp_line (start 0.25 0) (end -0.75 1)
+      (stroke (width 0.3) (type solid)) (layer "Dwgs.User"))
+    (fp_line (start 0.25 1) (end 0.25 -1)
+      (stroke (width 0.3) (type solid)) (layer "Dwgs.User"))
+  )
+  (footprint "riotee:KikitTab" (layer "F.Cu")
+    (at 223.86 50.55 -90)
+    (descr "A symbol representing annotation for tab placement")
+    (attr exclude_from_pos_files exclude_from_bom)
+    (fp_text reference "REF**" (at 0 -2 90) (layer "F.SilkS") hide
+        (effects (font (size 1 1) (thickness 0.15)))
+    )
+    (fp_text value "Tab" (at -2.75 -1 90) (layer "Dwgs.User")
+        (effects (font (size 1.2 1.2) (thickness 0.2)))
+    )
+    (fp_text user "KIKIT: width: 3mm" (at -5.5 0) (layer "Dwgs.User")
+        (effects (font (size 1 1) (thickness 0.15)))
+    )
+    (fp_line (start 0.25 0) (end -2.75 0)
+      (stroke (width 0.3) (type solid)) (layer "Dwgs.User"))
+    (fp_line (start 0.25 0) (end -0.75 -1)
+      (stroke (width 0.3) (type solid)) (layer "Dwgs.User"))
+    (fp_line (start 0.25 0) (end -0.75 1)
+      (stroke (width 0.3) (type solid)) (layer "Dwgs.User"))
+    (fp_line (start 0.25 1) (end 0.25 -1)
+      (stroke (width 0.3) (type solid)) (layer "Dwgs.User"))
+  )
+  (footprint "riotee:KikitTab" (layer "F.Cu")
+    (at 233.93 62.23 180)
+    (descr "A symbol representing annotation for tab placement")
+    (attr exclude_from_pos_files exclude_from_bom)
+    (fp_text reference "REF**" (at 0 -2) (layer "F.SilkS") hide
+        (effects (font (size 1 1) (thickness 0.15)))
+    )
+    (fp_text value "Tab" (at -2.75 -1) (layer "Dwgs.User")
+        (effects (font (size 1.2 1.2) (thickness 0.2)))
+    )
+    (fp_text user "KIKIT: width: 3mm" (at -5.5 0 90) (layer "Dwgs.User")
+        (effects (font (size 1 1) (thickness 0.15)))
+    )
+    (fp_line (start 0.25 0) (end -2.75 0)
+      (stroke (width 0.3) (type solid)) (layer "Dwgs.User"))
+    (fp_line (start 0.25 0) (end -0.75 -1)
+      (stroke (width 0.3) (type solid)) (layer "Dwgs.User"))
+    (fp_line (start 0.25 0) (end -0.75 1)
+      (stroke (width 0.3) (type solid)) (layer "Dwgs.User"))
+    (fp_line (start 0.25 1) (end 0.25 -1)
+      (stroke (width 0.3) (type solid)) (layer "Dwgs.User"))
+  )
   (footprint "riotee:AS_KXOB25_23x08" (layer "F.Cu")
     (at 183.1 62.23 90)
@@
       (rotate (xyz 0 0 180))
     )
+  )
+  (footprint "riotee:KikitTab" (layer "F.Cu")
+    (at 177.55 62.23)
+    (descr "A symbol representing annotation for tab placement")
+    (attr exclude_from_pos_files exclude_from_bom)
+    (fp_text reference "REF**" (at 0 -2) (layer "F.SilkS") hide
+        (effects (font (size 1 1) (thickness 0.15)))
+    )
+    (fp_text value "Tab" (at -2.75 -1) (layer "Dwgs.User")
+        (effects (font (size 1.2 1.2) (thickness 0.2)))
+    )
+    (fp_text user "KIKIT: width: 3mm" (at -5.5 0 90) (layer "Dwgs.User")
+        (effects (font (size 1 1) (thickness 0.15)))
+    )
+    (fp_line (start 0.25 0) (end -2.75 0)
+      (stroke (width 0.3) (type solid)) (layer "Dwgs.User"))
+    (fp_line (start 0.25 0) (end -0.75 -1)
+      (stroke (width 0.3) (type solid)) (layer "Dwgs.User"))
+    (fp_line (start 0.25 0) (end -0.75 1)
+      (stroke (width 0.3) (type solid)) (layer "Dwgs.User"))
+    (fp_line (start 0.25 1) (end 0.25 -1)
+      (stroke (width 0.3) (type solid)) (layer "Dwgs.User"))
   )
   (footprint "riotee:TE_1825058-1" (layer "F.Cu")
@@
     )
   )
+  (footprint "riotee:KikitTab" (layer "F.Cu")
+    (at 223.86 73.91 90)
+    (descr "A symbol representing annotation for tab placement")
+    (attr exclude_from_pos_files exclude_from_bom)
+    (fp_text reference "REF**" (at 0 -2 90) (layer "F.SilkS") hide
+        (effects (font (size 1 1) (thickness 0.15)))
+    )
+    (fp_text value "Tab" (at -2.75 -1 90) (layer "Dwgs.User")
+        (effects (font (size 1.2 1.2) (thickness 0.2)))
+    )
+    (fp_text user "KIKIT: width: 3mm" (at -5.5 0) (layer "Dwgs.User")
+        (effects (font (size 1 1) (thickness 0.15)))
+    )
+    (fp_line (start 0.25 0) (end -2.75 0)
+      (stroke (width 0.3) (type solid)) (layer "Dwgs.User"))
+    (fp_line (start 0.25 0) (end -0.75 -1)
+      (stroke (width 0.3) (type solid)) (layer "Dwgs.User"))
+    (fp_line (start 0.25 0) (end -0.75 1)
+      (stroke (width 0.3) (type solid)) (layer "Dwgs.User"))
+    (fp_line (start 0.25 1) (end 0.25 -1)
+      (stroke (width 0.3) (type solid)) (layer "Dwgs.User"))
+  )
   (footprint "riotee:AS_KXOB25_23x08" (layer "F.Cu")
